Commit message: fixed the joint 2

File: task4ws/arm_description/urdf/arm.urdf (robot description, URDF)
Before this commit: robot Ufactoryufactory-xarm-lite-6, 8 links, 7 joints
Joints:
- joint joint_1: origin xyz=0.0 0.0 0.2 rpy=0.0 0.0 0.0 -> xyz=0.0 0.0 0.24 rpy=0.0 0.0 0.0; type revolute -> continuous
- joint joint_2: axis 0.0 0.0 1.0 -> 0.0 0.0 0.1; origin xyz=0.0 0.012 0.2 rpy=0.0 0.0 0.0 -> xyz=0.0 -0.001 -0.001 rpy=-1.57 -1.57 0.0
- joint joint_3: axis 0.0 1.0 0.0 -> 0.0 0.0 0.1; origin xyz=0.0 0.03 0.0 rpy=0.0 0.0 0.0 -> xyz=0.2 -0.001 0.01 rpy=-3.2 0.0 0.0
- joint joint_4: axis 0.0 0.0 1.0 -> 0.0 1.0 0.0; origin xyz=0.10 0.011 -0.220 rpy=0.0 0.0 0.0 -> xyz=0.09 -0.227 -0.004 rpy=0.0 0.0 0.0
- joint joint_5: origin xyz=0.0 0.0 0.00 rpy=0.0 3.14 3.14 -> xyz=0.0 0.0 0.00 rpy=1.57 3.14 0.0
